File: tests/test_arc.kicad_pcb (KiCad board)
At the start: 2 copper layers, 0 parts

Commit message: more tests
Other:
- board text added: "CW"
- board text added: "CW hm"

Commit message: add more arc tests
Other:
- board text added: "CCW"
- board text added: "CW vm"
