File: tests/test_text.kicad_pcb (KiCad board)
At the start: 2 copper layers, 0 parts

Commit message: add more text tests, work on vertical alignment
Other:
- board text added: "line1 Line 2 lin3"
- board text removed: "Thres Pre/Post"
- board text removed: "t/Div Samples"
Changed lines of the file:
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@@
+	)
+	(gr_line
+		(start 103.2 78.8)
+		(end 146.8 78.8)
+		(stroke
+			(width 0.1)
+			(type default)
+		)
+		(layer "User.3")
+	)
+	(gr_line
+		(start 103.2 92.9)
+		(end 103.2 78.8)
+		(stroke
+			(width 0.1)
+			(type default)
+		)
+		(layer "User.3")
 	)
 	(gr_line
@@
 	)
 	(gr_line
+		(start 131 92.9)
+		(end 131.2 92.9)
+		(stroke
+			(width 0.1)
+			(type default)
+		)
+		(layer "User.3")
+	)
+	(gr_line
 		(start 131.2 65.1)
 		(end 131.2 74.3)
@@
 		(start 145 74.3)
 		(end 103.2 74.3)
+		(stroke
+			(width 0.1)
+			(type default)
+		)
+		(layer "User.3")
+	)
+	(gr_line
+		(start 146.8 78.8)
+		(end 146.8 93)
+		(stroke
+			(width 0.1)
+			(type default)
+		)
+		(layer "User.3")
+	)
+	(gr_line
+		(start 146.8 93)
+		(end 103.2 92.9)
 		(stroke
 			(width 0.1)
@@
 	)
 	(gr_text "Range\nOfs"
-		(at 144.4 85.1 0)
+		(at 144.1 114.1 0)
 		(layer "User.4")
 		(effects
@@
 		)
 	)
-	(gr_text "Range\nOfs"
-		(at 111.2 84.3 0)
+	(gr_text "line1\nLine 2\nlin3"
+		(at 139.4 79.4 0)
+		(layer "User.4" knockout)
+		(effects
+			(font
+				(size 3 3)
+				(thickness 0.5)
+			)
+			(justify top)
+		)
+	)
+	(gr_text "Range\nOfs"
+		(at 110.9 113.3 0)
 		(layer "User.4")
 		(effects
@@
 		)
 	)
-	(gr_text "Range\nOfs"
-		(at 135.7 96.5 0)
+	(gr_text "line1\nLine 2\nlin3"
+		(at 124.8 86 0)
 		(layer "User.4" knockout)
 		(effects
@@
 		)
 	)
-	(gr_text "Range\nOfs"
-		(at 112.86 107.8 0)
-		(layer "User.4")
+	(gr_text "line1\nLine 2\nlin3"
+		(at 110.3 92.6 0)
+		(layer "User.4" knockout)
 		(effects
 			(font
@@
 		)
 	)
-	(gr_text "t/Div\nSamples"
-		(at 154.36 108.8 0)
-		(layer "User.4")
-		(effects
-			(font
-				(size 3 3)
-				(thickness 0.5)
-			)
-			(justify bottom)
-		)
-	)
 	(gr_text "Mode"
 		(at 120.9 51.2 0)
@@
 		)
 	)
-	(gr_text "Thres\nPre/Post"
-		(at 130.4 116.4 0)
-		(layer "User.4")
-		(effects
-			(font
-				(size 3 3)
-				(thickness 0.5)
-			)
-			(justify right bottom)
-		)
-	)
-	(gr_text "Range\nOfs"
-		(at 127.8 84.6 0)
+	(gr_text "Range\nOfs"
+		(at 127.5 113.6 0)
 		(layer "User.4")
 		(effects
@@
 	)
 	(gr_text "Range\nOfs"
-		(at 160.9 85.1 0)
-		(layer "User.4")
-		(effects
+		(at 160.6 114.1 0)
+		(layer "User.4")
+		(effects

Commit message: add more text tests for mirrored, rotated text, remove old comment
Other:
- board text added: "rotated"
- board text added: "rotated+ mirrored"
- board text removed: "Mode"
Changed lines of the file:
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@@
-		)
-	)
-	(gr_text "Mode"
-		(at 108.9 43.4 0)
-		(layer "User.4")
-		(effects
-			(font
-				(size 3 3)
-				(thickness 0.5)
-			)
-			(justify left bottom)
 		)
 	)
@@
 			)
 			(justify top)
+		)
+	)
+	(gr_text "Range\nOfs"
+		(at 144 55.3 0)
+		(layer "User.4" knockout)
+		(effects
+			(font
+				(size 3 3)
+				(thickness 0.5)
+			)
+			(justify top)
+		)
+	)
+	(gr_text "line1\nLine 2\nlin3"
+		(at 158.6 80.2 0)
+		(layer "User.4" knockout)
+		(effects
+			(font
+				(size 3 3)
+				(thickness 0.5)
+			)
+			(justify top)
+		)
+	)
+	(gr_text "Range\nOfs"
+		(at 143.8 40.7 0)
+		(layer "User.4" knockout)
+		(effects
+			(font
+				(size 3 3)
+				(thickness 0.5)
+			)
+			(justify top mirror)
 		)
 	)
@@
 		)
 	)
+	(gr_text "rotated+\nmirrored"
+		(at 160.2 45.8 0)
+		(layer "User.4")
+		(effects
+			(font
+				(size 3 3)
+				(thickness 0.5)
+			)
+		)
+	)
+	(gr_text "rotated"
+		(at 160.4 59.4 0)
+		(layer "User.4")
+		(effects
+			(font
+				(size 3 3)
+				(thickness 0.5)
+			)
+		)
+	)
 	(gr_text "Range\nOfs"
 		(at 110 74 0)
@@
 		)
 	)
-	(gr_text "Mode"
-		(at 114.9 47.3 0)
-		(layer "User.4")
+	(gr_text "Range\nOfs"
+		(at 103.7 57.2 90)
+		(layer "User.4" knockout)
 		(effects
 			(font
@@
 				(thickness 0.5)
 			)
-			(justify bottom)
+			(justify top)
 		)
 	)
-	(gr_text "Mode"
-		(at 120.9 51.2 0)
-		(layer "User.4")
+	(gr_text "Range\nOfs"
+		(at 103.5 42.6 90)
+		(layer "User.4" knockout)
 		(effects
 			(font
@@
 				(thickness 0.5)
 			)
-			(justify right bottom)
+			(justify top mirror)
 		)
 	)
+	(gr_text "Range\nOfs"
+		(at 120.1 63.5 180)
+		(layer "User.4" knockout)
+		(effects
+			(font
+				(size 3 3)
+				(thickness 0.5)
+			)
+			(justify top)
+		)
+	)
+	(gr_text "Range\nOfs"
+		(at 119.9 48.9 180)
+		(layer "User.4" knockout)
+		(effects
+			(font
+				(size 3 3)
+				(thickness 0.5)
+			)
+			(justify top mirror)
+		)
+	)
+	(gr_text "Range\nOfs"
+		(at 136.2 57 270)
+		(layer "User.4" knockout)
+		(effects
+			(font
+				(size 3 3)
+				(thickness 0.5)
+			)
+			(justify top)
+		)
+	)
+	(gr_text "Range\nOfs"
+		(at 136 42.4 270)
+		(layer "User.4" knockout)
+		(effects
+			(font
+				(size 3 3)
+				(thickness 0.5)
+			)
+			(justify top mirror)
+		)
+	)

Commit message: add vertical alignment test for single lines of text
Other:
- board text added: "testXX"
- board text added: "vbot"
- board text added: "vmid"
- board text added: "vtop"
Changed lines of the file:
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@@
+	)
+	(gr_line
+		(start 102.55 98.75)
+		(end 147 98.75)
+		(stroke
+			(width 0.1)
+			(type default)
+		)
+		(layer "User.3")
+	)
+	(gr_line
+		(start 102.55 103.1)
+		(end 102.55 98.75)
+		(stroke
+			(width 0.1)
+			(type default)
+		)
+		(layer "User.3")
 	)
 	(gr_line
@@
 	)
 	(gr_line
+		(start 117.3 98.75)
+		(end 117.3 103.05)
+		(stroke
+			(width 0.1)
+			(type default)
+		)
+		(layer "User.3")
+	)
+	(gr_line
+		(start 117.4 98.75)
+		(end 117.4 103.05)
+		(stroke
+			(width 0.1)
+			(type default)
+		)
+		(layer "User.3")
+	)
+	(gr_line
 		(start 131 65.1)
 		(end 131 74.3)
@@
 	)
 	(gr_line
+		(start 132.15 98.75)
+		(end 132.15 103.05)
+		(stroke
+			(width 0.1)
+			(type default)
+		)
+		(layer "User.3")
+	)
+	(gr_line
+		(start 132.25 98.75)
+		(end 132.25 103.05)
+		(stroke
+			(width 0.1)
+			(type default)
+		)
+		(layer "User.3")
+	)
+	(gr_line
 		(start 145 65)
 		(end 145 74.3)
@@
 		(start 146.8 93)
 		(end 103.2 92.9)
+		(stroke
+			(width 0.1)
+			(type default)
+		)
+		(layer "User.3")
+	)
+	(gr_line
+		(start 147 98.75)
+		(end 147 103.05)
+		(stroke
+			(width 0.1)
+			(type default)
+		)
+		(layer "User.3")
+	)
+	(gr_line
+		(start 147 103.05)
+		(end 102.55 103.1)
 		(stroke
 			(width 0.1)
@@
 	)
 	(gr_text "Range\nOfs"
-		(at 144.1 114.1 0)
+		(at 144.15 115.15 0)
 		(layer "User.4")
 		(effects
@@
 		)
 	)
+	(gr_text "testXX"
+		(at 110 99.3 0)
+		(layer "User.4" knockout)
+		(effects
+			(font
+				(size 3 3)
+				(thickness 0.5)
+			)
+			(justify top)
+		)
+	)
+	(gr_text "vtop"
+		(at 110.1 104 0)
+		(layer "User.4")
+		(effects
+			(font
+				(size 3 3)
+				(thickness 0.5)
+			)
+			(justify top)
+		)
+	)
+	(gr_text "vmid"
+		(at 125.05 104.1 0)
+		(layer "User.4")
+		(effects
+			(font
+				(size 3 3)
+				(thickness 0.5)
+			)
+			(justify top)
+		)
+	)
 	(gr_text "Range\nOfs"
 		(at 138 65.6 0)
@@
 		)
 	)
+	(gr_text "vbot"
+		(at 139.55 103.95 0)
+		(layer "User.4")
+		(effects
+			(font
+				(size 3 3)
+				(thickness 0.5)
+			)
+			(justify top)
+		)
+	)
 	(gr_text "Range\nOfs"
 		(at 144 55.3 0)
@@
 	)
 	(gr_text "Range\nOfs"
-		(at 110.9 113.3 0)
+		(at 110.95 114.35 0)
 		(layer "User.4")
 		(effects
@@
 		)
 	)
+	(gr_text "testXX"
+		(at 124.85 101.05 0)
+		(layer "User.4" knockout)
+		(effects
+			(font
+				(size 3 3)
+				(thickness 0.5)
+			)
+		)
+	)
 	(gr_text "rotated+\nmirrored"
 		(at 160.2 45.8 0)
@@
 		)
 	)
+	(gr_text "testXX"
+		(at 139.7 102.8 0)
+		(layer "User.4" knockout)
+		(effects
+			(font
+				(size 3 3)
+				(thickness 0.5)
+			)
+			(justify bottom)
+		)
+	)
 	(gr_text "Range\nOfs"
 		(at 103.7 57.2 90)
@@
 	)
 	(gr_text "Range\nOfs"
-		(at 127.5 113.6 0)
+		(at 127.55 114.65 0)
 		(layer "User.4")
 		(effects
@@
 	)
 	(gr_text "Range\nOfs"
-		(at 160.6 114.1 0)
-		(layer "User.4")
-		(effects
+		(at 160.65 115.15 0)
+		(layer "User.4")
+		(effects

Commit message: add horizontal alignment tests for text
Other:
- board text added: "hl"
- board text added: "hmid"
- board text added: "hr"
