File: tests/test_text.kicad_pcb (KiCad board)
At the start: 2 copper layers, 0 parts

Commit message: read font face from KiCad text if present
Other:
- board text added: "f:Carlito"

Commit message: add valign test for text with 4 lines
Other:
- board text added: "line1 Line 2 lin3 line4"
