File: tests/test_text.kicad_pcb (KiCad board)
At the start: 2 copper layers, 0 parts

Commit message: Add a bit of naughtiness to the text test 8-) (nasty chars & HTML/JS injection attempt)
Other:
- board text added: "<script>alert({dblquote}fail!{dblquote});</script>"
- board text added: "{} ! '' `` '' \t \ \\"
Changed lines of the file:
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@@
+		)
+	)
+	(gr_text "<script>alert({dblquote}fail!{dblquote});</script>"
+		(at 102.2 119 0)
+		(layer "User.4")
+		(effects
+			(font
+				(size 1 1)
+				(thickness 0.15)
+			)
+			(justify left bottom)
+		)
+	)
+	(gr_text "{} ! '' `` ''	 \\t \\ \\\\ "
+		(at 127.6 119 0)
+		(layer "User.4")
+		(effects
+			(font
+				(size 1 1)
+				(thickness 0.15)
+			)
+			(justify left bottom)
 		)
 	)
