File: tests/test_layers.kicad_pcb (KiCad board)
At the start: 2 copper layers, 0 parts

Commit message: test_layers: make texts distinguishable from each other
Other:
- board text added: "Test456"
Changed lines of the file:
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@@
 		(layer "User.4")
 	)
-	(gr_text "Test123"
+	(gr_text "Test456"
 		(at 145 105 0)
 		(layer "User.3")

Commit message: add another test text in F.Mask
Other:
- board text added: "TestABC"
Changed lines of the file:
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@@
 		(layer "User.4")
+	)
+	(gr_text "TestABC"
+		(at 128 82 0)
+		(layer "User.2")
+		(effects
+			(font
+				(size 5 5)
+				(bold yes)
+			)
+			(justify left bottom)
+		)
 	)
 	(gr_text "Test456"
